File: Non-Prog/KiCAD/Non-Programmable Throttle Control.sch (KiCad schematic (older format))
At the start: 14 parts, among them P1 CONN_01X06, U1 LM2902N, U2 LM555N

Commit message: Updated Details, Added pinout to schematic
Parts:
- removed JP1: JUMPER3, symbol JUMPER3
- removed unit 4 of U1
- C1: value 1uF -> C; footprint (none) -> Capacitors_SMD:C_0603
- D1: value D_Schottky_x2_Serial_AKC -> DA3X101F0L; footprint (none) -> TO_SOT_Packages_SMD:SOT-23
- P1: footprint (none) -> Pin_Headers:Pin_Header_Straight_1x06
- R1, R2, R3, R4, R5, R7, R8: footprint (none) -> Resistors_SMD:R_0603
- R6: value 1k -> 2.2k; footprint (none) -> Resistors_SMD:R_0603
- U1: value LM2902N -> LM324ADR; footprint (none) -> Housings_SOIC:SOIC-14_3.9x8.7mm_Pitch1.27mm
- U2: footprint (none) -> Housings_SOIC:SOIC-8_3.9x4.9mm_Pitch1.27mm
Connections:
- wire segments 73 -> 86
Other:
- note added: "RPI FSAE\nNon-Programmable\nElectronic Throttle Safety Interlock System\n\nRevised: 2/20/2016\n\nPinout:\n1-Input 1 (Brake Press/TPS)\n2-Input 2 (Brake Press/TPS)\n3-VCC\n4-Output\n5-Connection to car start button\n6-Ground"
