File: Non-Prog/KiCAD/NetListNonProg.kicad_pcb (KiCad board)
At the start: 2 copper layers, 25 x 25 mm, 15 parts, among them P1 CONN_01X06, U1 LM324ADR, U2 555

Commit message: Updated PCB Files
Parts:
- R4, R5, R6, R7, U2: moved to F.Cu
- moved U2 7.08 mm to (143.7, 78.8), turned to 270 degrees
- moved R7 5.50 mm to (145.2, 83.5), turned to 0 degrees
- moved R8 4.83 mm to (138.3, 81.9), turned to 270 degrees
- moved R4 4.47 mm to (133.5, 84.9)
- moved R5 4.43 mm to (131.3, 84.4), turned to 0 degrees
- moved R6 4.37 mm to (135.4, 84.9)
- moved R1 3.69 mm to (129.1, 75.5)
- moved R3 3.64 mm to (129.1, 82.2)
- moved D1 3.63 mm to (139.2, 78.8)
- moved C1 3.63 mm to (139.0, 76.4)
- moved R2 3.63 mm to (129.1, 78.8)
- moved U1 3.63 mm to (133.7, 78.8)
Routing:
- net GND: track 44.4 -> 57.9 mm, vias 2 -> 1
- net VCC: track 25.8 -> 33.3 mm, vias 1 -> 0
- net Net-(R4-Pad2): track 7.10 -> 10.7 mm, vias 1 -> 0
- net Net-(R2-Pad2): track 6.62 -> 3.80 mm
- net Net-(R1-Pad2): track 6.59 -> 3.84 mm
- net Net-(P1-Pad2): track 10.3 -> 8.31 mm
- net Net-(P1-Pad5): track 8.38 -> 6.51 mm
- net Net-(P1-Pad1): track 12.9 -> 11.3 mm
- net Net-(C1-Pad1): track 6.13 -> 7.69 mm, vias 1 -> 0
- net Net-(R6-Pad2): track 13.7 -> 15.1 mm, vias 1 -> 0
- net Net-(P1-Pad4): track 6.27 -> 7.04 mm
- net Net-(R4-Pad1): track 8.43 -> 9.18 mm, vias 1 -> 0
- net Net-(R5-Pad1): track 2.50 -> 1.95 mm, vias 1 -> 0
